File: plates/pcb/bottom/corne-bottom-plate.kicad_pcb (KiCad board)
At the start: 2 copper layers, 133.8 x 91.4 mm, 7 parts

Commit message: minor improvements in tracing
Other:
- rule pad_to_mask_clearance: 0.2 -> 0
