File: plates/pcb/top/corne-top-plate.kicad_pcb (KiCad board)
At the start: 2 copper layers, 132.9 x 91.4 mm, 28 parts, among them SW2 KEY_SWITCH

Commit message: minor improvements in tracing
Other:
- rule pad_to_mask_clearance: 0.2 -> 0
